File: Kicad/mosaicG5 HAT/mosaicG5_RPi_HAT.kicad_sch (KiCad schematic)
At the start: 54 parts, among them J1 Conn_01x02_Pin, J10 Conn_Coaxial, J11 Conn_Coaxial, J12 Conn_Coaxial, J13 Conn_01x06_Pin, J14 Conn_Coaxial, J2 Conn_01x05_Pin, J3 USB4105-GF-A, U1 mosaic-G5, U10 XC8111AA01MR-G, U2 ECMF02-2AMX6, U3 MP2145GD-Z, U4 TPS7A9401DSCR, U5 XC8111AA01MR-G, U9 XC8111AA01MR-G

Commit message: logo schematic
Other:
- note added: "Designed By: Laetitia.KF"
Changed lines of the file:
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@@
+		)
+	)
+	(text "Designed By: Laetitia.KF"
+		(exclude_from_sim no)
+		(at 391.16 276.86 0)
+		(effects
+			(font
+				(size 1.27 1.27)
+				(color 132 0 0 1)
+			)
 		)
 	)
